Commit message: Removed stage, fixed gazebo simulation

File: xacro/p3dx/pioneer3dx.xacro (robot description, xacro)
@@ -2,11 +2,11 @@
 <robot xmlns:xacro="http://ros.org/wiki/xacro" name="pioneer3dx" >
   <!-- Import Rviz colors -->
-  <xacro:include filename="$(find gazebo_plugins)/test/multi_robot_scenario/xacro/materials.xacro" />
+  <xacro:include filename="$(find pioneer3dx)/xacro/materials.xacro" />
   <!-- Import robot -->
   <xacro:include filename="$(find pioneer3dx)/xacro/p3dx/pioneer3dx_body.xacro"/>
-  <xacro:pioneer3dx_body name="chassis" parent="base_link" meshes="package://gazebo_plugins/test/multi_robot_scenario/meshes/p3dx"/>
+  <xacro:pioneer3dx_body name="chassis" parent="base_link" meshes="package://pioneer3dx/meshes/p3dx"/>
   <!-- Laser  -->
   <xacro:include filename="$(find pioneer3dx)/xacro/laser/hokuyo.xacro"/>
-  <xacro:laser name="front_laser" parent="chassis" xyz="0.0 0 0.26" rpy="0 0 0" meshes="package://gazebo_plugins/test/multi_robot_scenario/meshes/"/>
+  <xacro:laser name="front_laser" parent="chassis" xyz="0.0 0 0.26" rpy="0 0 0" meshes="package://pioneer3dx/meshes/"/>
   <!-- Sonar
   <xacro:include filename="$(find pioneer3dx)/xacro/p3dx/pioneer3dx_sonar.xacro" />

File: xacro/p3dx/pioneer3dx_sonar.xacro (robot description, xacro)
@@ -27,5 +27,5 @@
       <origin xyz="0 0 0" rpy="0 0 0"/>
       <geometry>
-        <box size="0 0 0"/>
+        <box size="0.1 0.1 0.1"/>
       </geometry>
     </collision>

File: xacro/p3dx/pioneer3dx_swivel.xacro (robot description, xacro)
@@ -31,5 +31,5 @@
       <origin xyz="0 0 0" rpy="0 0 0"/>
       <geometry>
-        <box size="0 0 0"/>
+        <box size="0.1 0.1 0.1"/>
       </geometry>
     </collision>
@@ -98,5 +98,5 @@
       <origin xyz="0 0 0" rpy="0 0 0"/>
       <geometry>
-        <box size="0 0 0"/>
+        <box size="0.1 0.1 0.1"/>
       </geometry>
     </collision>

File: xacro/p3dx/pioneer3dx_wheel.xacro (robot description, xacro)
@@ -29,5 +29,5 @@
       <origin xyz="0 0 0" rpy="0 0 0"/>
       <geometry>
-        <box size="0 0 0"/>
+        <box size="0.1 0.1 0.1"/>
       </geometry>
     </collision>
